Commit message: added most attempts

File: xacro/description.urdf.xacro (robot description, xacro)
@@ -5,4 +5,5 @@
 >
 	<xacro:include filename="$(find ros_indigo_urdf_gazebo_ogre)/xacro/link_joint.urdf.xacro"/>
+	<xacro:include filename="$(find ros_indigo_urdf_gazebo_ogre)/xacro/link_joint_dae.urdf.xacro"/>
 	<link name="link_origin"/>
 	<link name="link_0">
@@ -31,6 +32,6 @@
 	</link>
 	<joint
-	    name="joint_0"
-	    type="fixed"
+		name="joint_0"
+		type="fixed"
 	>
 		<origin xyz="0 0 0.00915298218"/>
@@ -38,15 +39,29 @@
 		<child link="link_0"/>
 	</joint>
-	<xacro:link_joint_macro
-		name="1"
-		parent="0"
+	<xacro:link_joint_macro name="1"/>
+	<xacro:link_joint_macro name="2"/>
+	<xacro:link_joint_macro name="3"/>
+	<xacro:link_joint_macro name="4"/>
+	<xacro:link_joint_macro name="5"/>
+	<xacro:link_joint_macro name="6"/>
+	<xacro:link_joint_macro name="7"/>
+	<xacro:link_joint_macro name="8"/>
+	<xacro:link_joint_macro name="9"/>
+	<xacro:link_joint_macro name="10"/>
+	<xacro:link_joint_macro name="11"/>
+	<xacro:link_joint_macro name="12"/>
+	<xacro:link_joint_macro name="13"/>
+	<xacro:link_joint_macro name="14"/>
+	<xacro:link_joint_macro name="15"/>
+	<xacro:link_joint_macro name="16"/>
+	<xacro:link_joint_macro name="17"/>
+	<xacro:link_joint_macro name="18"/>
+	<xacro:link_joint_dae_macro
+		name="19"
+		mesh="dodecahedron_ambient_0.dae"
 	/>
-	<xacro:link_joint_macro
-		name="2"
-		parent="1"
-	/>
-	<xacro:link_joint_macro
-		name="3"
-		parent="2"
+	<xacro:link_joint_dae_macro
+		name="20"
+		mesh="dodecahedron_ambient_1.dae"
 	/>
 	<gazebo reference="link_1">
@@ -59,3 +74,62 @@
 		<material>ros_indigo_urdf_gazebo_ogre/Azure</material>
 	</gazebo>
+	<gazebo reference="link_4"><material><script>
+		<uri>file://media/materials/scripts/gazebo.material</uri>
+		<name>ros_indigo_urdf_gazebo_ogre/Azure</name>
+	</script></material></gazebo>
+	<gazebo reference="link_5"><material><script>
+		<uri>file://media/materials/scripts/ros_indigo_urdf_gazebo_ogre.material</uri>
+		<name>ros_indigo_urdf_gazebo_ogre/Azure</name>
+	</script></material></gazebo>
+	<gazebo reference="link_6"><material><script>
+		<uri>file://Media/materials/scripts/ros_indigo_urdf_gazebo_ogre.material</uri>
+		<name>ros_indigo_urdf_gazebo_ogre/Azure</name>
+	</script></material></gazebo>
+	<gazebo reference="link_7"><material><script>
+		<uri>file://materials/scripts/ros_indigo_urdf_gazebo_ogre.material</uri>
+		<name>ros_indigo_urdf_gazebo_ogre/Azure</name>
+	</script></material></gazebo>
+	<gazebo reference="link_8"><material><script>
+		<uri>file://scripts/ros_indigo_urdf_gazebo_ogre.material</uri>
+		<name>ros_indigo_urdf_gazebo_ogre/Azure</name>
+	</script></material></gazebo>
+	<gazebo reference="link_9"><material><script>
+		<uri>file://ros_indigo_urdf_gazebo_ogre.material</uri>
+		<name>ros_indigo_urdf_gazebo_ogre/Azure</name>
+	</script></material></gazebo>
+	<gazebo reference="link_10"><material><script>
+		<uri>file://home/guir/catkin_ws/src/ros_indigo_urdf_gazebo_ogre/media/materials/scripts/ros_indigo_urdf_gazebo_ogre.material</uri>
+		<name>ros_indigo_urdf_gazebo_ogre/Azure</name>
+	</script></material></gazebo>
+	<gazebo reference="link_11"><material><script>
+		<uri>file://home/guir/catkin_ws/src/ros_indigo_urdf_gazebo_ogre/Media/materials/scripts/ros_indigo_urdf_gazebo_ogre.material</uri>
+		<name>ros_indigo_urdf_gazebo_ogre/Azure</name>
+	</script></material></gazebo>
+	<gazebo reference="link_12"><material><script>
+		<uri>file://home/guir/catkin_ws/src/ros_indigo_urdf_gazebo_ogre/media/materials/ros_indigo_urdf_gazebo_ogre.material</uri>
+		<name>ros_indigo_urdf_gazebo_ogre/Azure</name>
+	</script></material></gazebo>
+	<gazebo reference="link_13"><material><script>
+		<uri>file://home/guir/catkin_ws/src/ros_indigo_urdf_gazebo_ogre/Media/materials/ros_indigo_urdf_gazebo_ogre.material</uri>
+		<name>ros_indigo_urdf_gazebo_ogre/Azure</name>
+	</script></material></gazebo>
+	<gazebo reference="link_14"><material><script>
+		<uri>file://home/guir/catkin_ws/src/ros_indigo_urdf_gazebo_ogre/media/ros_indigo_urdf_gazebo_ogre.material</uri>
+		<name>ros_indigo_urdf_gazebo_ogre/Azure</name>
+	</script></material></gazebo>
+	<gazebo reference="link_15"><material><script>
+		<uri>file://home/guir/catkin_ws/src/ros_indigo_urdf_gazebo_ogre/Media/ros_indigo_urdf_gazebo_ogre.material</uri>
+		<name>ros_indigo_urdf_gazebo_ogre/Azure</name>
+	</script></material></gazebo>
+	<gazebo reference="link_16"><material><script>
+		<uri>file://home/guir/catkin_ws/src/ros_indigo_urdf_gazebo_ogre/ros_indigo_urdf_gazebo_ogre.material</uri>
+		<name>ros_indigo_urdf_gazebo_ogre/Azure</name>
+	</script></material></gazebo>
+	<gazebo reference="link_17"><material><script>
+		<uri>file:///home/guir/catkin_ws/src/ros_indigo_urdf_gazebo_ogre/ros_indigo_urdf_gazebo_ogre.material</uri>
+		<name>ros_indigo_urdf_gazebo_ogre/Azure</name>
+	</script></material></gazebo>
+	<gazebo reference="link_18">
+		<material>ros_indigo_urdf_gazebo_ogre.material</material>
+	</gazebo>
 </robot>

File: xacro/link_joint_dae.urdf.xacro (robot description, xacro)
@@ -2,6 +2,6 @@
 <robot xmlns:xacro="http://www.ros.org/wiki/xacro">
 	<xacro:macro
-		name="link_joint_macro"
-		params="name"
+		name="link_joint_dae_macro"
+		params="name mesh"
 	>
 	    <link name="link_${name}">
@@ -20,10 +20,10 @@
                     <visual>
                             <geometry>
-                                    <mesh filename="package://ros_indigo_urdf_gazebo_ogre/mesh/dodecahedron.STL"/>
+                                    <mesh filename="package://ros_indigo_urdf_gazebo_ogre/mesh/${mesh}"/>
                             </geometry>
                     </visual>
                     <collision>
                             <geometry>
-                                    <mesh filename="package://ros_indigo_urdf_gazebo_ogre/mesh/dodecahedron.STL"/>
+                                    <mesh filename="package://ros_indigo_urdf_gazebo_ogre/mesh/${mesh}"/>
                             </geometry>
                     </collision>

Commit message: changed robot and image for better fit

File: xacro/description.urdf.xacro (robot description, xacro)
@@ -35,5 +35,8 @@
 		type="fixed"
 	>
-		<origin xyz="0 0 0.00915298218"/>
+		<origin
+			xyz="0 0 0.02"
+			rpy="0 1.570796 0"
+		/>
 		<parent link="link_origin"/>
 		<child link="link_0"/>
